File: PCB/fub.kicad_sch (KiCad schematic)
At the start: 36 parts, among them J2 SAMDfix, J8 Type-C_5077CR-16SMC2-BK-TR, SW1 SW_SPDT, U1 MS18F, U2 LM1117GS-3.3, U3 ATSAMD21G18A_ARM-Cortex-m0+, U4 AT24C32E-EEPROM, Y1 FC-135_32.7680KHz

Commit message: Add files via upload
Other:
- title: ark.*~ v.2 -> fub.*~
